Commit message: modified xacro files

File: robots/go1_description/xacro/robot.xacro (robot description, xacro)
@@ -17,5 +17,5 @@
         <link name="world"/>
         <joint name="base_static_joint" type="fixed">
-            <origin rpy="0 0 0" xyz="0 0 0"/>
+            <origin rpy="0 0 0" xyz="1 0 0.28"/>
             <parent link="world"/>
             <child link="base"/>
